File: kicad-pcb-01.kicad_pcb (KiCad board)
At the start: 2 copper layers, 77.8 x 38.1 mm, 24 parts, among them SW1 SW_Push, U1 ATmega32U4-AU, Y1 16MHz

Commit message: routing complete
Parts:
- moved C6 6.24 mm to (116.7, 130.7), turned to 270 degrees
- moved C4 0.16 mm to (131.8, 112.4)
- turned F1 to 90 degrees
- turned R3 to 270 degrees
Connections:
- U1 pad 26: Net-(U1-Pad26) -> ROW1
- U1 pad 27: Net-(U1-Pad27) -> ROW0
- U1 pad 28: Net-(U1-Pad28) -> COL1
- U1 pad 29: Net-(U1-Pad29) -> COL0
Routing:
- net GND: track 0.00 -> 137.3 mm
- net +5V: track 0.00 -> 104.4 mm, vias 0 -> 5
- net ROW1: track 0.00 -> 63.5 mm, vias 0 -> 2
- net ROW0: track 0.00 -> 54.9 mm
- net COL1: track 0.00 -> 53.0 mm
- net COL0: track 0.00 -> 32.7 mm
- net Net-(R3-Pad2): track 0.00 -> 32.6 mm, vias 0 -> 2
- net Net-(C5-Pad1): track 0.00 -> 31.4 mm, vias 0 -> 2
- net Net-(R1-Pad1): track 0.00 -> 23.0 mm
- net Net-(R2-Pad1): track 0.00 -> 22.4 mm
- net VCC: track 0.00 -> 13.2 mm
- net Net-(C4-Pad1): track 0.00 -> 10.5 mm
- net Net-(D1-Pad2): track 0.00 -> 7.23 mm
- net Net-(D3-Pad2): track 0.00 -> 7.23 mm
- net Net-(D4-Pad2): track 0.00 -> 7.03 mm
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Other:
- net class Default: trace_width 0.25 -> 0.254
- net class power added: clearance 0.2, trace_width 0.381, via_dia 0.8, via_drill 0.4

Commit message: complete
Routing:
- net Net-(USB1-Pad6): track 0.00 -> 22.2 mm
- added copper zone on B.Cu, net GND
Other:
- board text added: "panzerstadt, 20200711"
Changed lines of the file:
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@@
   (general
     (thickness 1.6)
-    (drawings 8)
-    (tracks 216)
+    (drawings 9)
+    (tracks 223)
     (zones 0)
     (modules 24)
@@
       (rotate (xyz 0 0 0))
     )
+  )
+  (gr_text "panzerstadt, 20200711" (at 128.5875 139.7) (layer F.SilkS)
+    (effects (font (size 1 1) (thickness 0.15)))
   )
   (gr_arc (start 100.80625 140.49375) (end 99.21875 140.49375) (angle -90) (layer Edge.Cuts) (width 0.05))
@@
   (segment (start 135.825 128.44375) (end 135.3325 128.93625) (width 0.254) (layer B.Cu) (net 20))
   (segment (start 136.525 128.44375) (end 135.825 128.44375) (width 0.254) (layer B.Cu) (net 20))
+  (segment (start 112.39375 105.56875) (end 110.33125 105.56875) (width 0.254) (layer B.Cu) (net 43))
+  (segment (start 105.09375 105.56875) (end 107.15625 105.56875) (width 0.254) (layer B.Cu) (net 43))
+  (segment (start 105.09375 110.06875) (end 105.09375 108.26875) (width 0.254) (layer B.Cu) (net 43))
+  (segment (start 112.39375 110.06875) (end 112.39375 108.425) (width 0.254) (layer B.Cu) (net 43))
+  (segment (start 112.39375 108.425) (end 112.39375 105.56875) (width 0.254) (layer B.Cu) (net 43))
+  (segment (start 105.09375 105.56875) (end 112.39375 105.56875) (width 0.254) (layer B.Cu) (net 43))
+  (segment (start 105.09375 105.56875) (end 105.09375 110.06875) (width 0.254) (layer B.Cu) (net 43))
+  (zone (net 1) (net_name GND) (layer B.Cu) (hatch edge 0.508)
+    (connect_pads (clearance 0.508))
+    (min_thickness 0.254)
+    (fill yes (arc_segments 32) (thermal_gap 0.508) (thermal_bridge_width 0.508) (smoothing fillet))
+    (polygon
+      (pts
+        (xy 138.90625 142.08125) (xy 99.21875 142.08125) (xy 99.21875 103.98125) (xy 138.90625 103.98125)
+      )
+    )
+  )
 )
